File: hw/pwrsupply.sch (KiCad schematic (older format))
At the start: 21 parts

Commit message: lots of changes, redesigning most of the PCB
Parts:
- removed D?: MUR160, Diode_THT:D_DO-15_P12.70mm_Horizontal, symbol Device:D
- removed U?: MC34063AP, Package_DIP:DIP-8_W7.62mm, symbol Regulator_Switching:MC34063AP
- added D2: MUR160, Diode_SMD:D_SMA-SMB_Universal_Handsoldering, symbol Diode:MRA4005T3G
- added U33: MC34063AD, Package_SO:SOIC-8_3.9x4.9mm_P1.27mm, symbol Regulator_Switching:MC34063AD
- L1: renamed from L?; footprint Inductor_THT:L_Radial_D8.7mm_P5.00mm_Fastron_07HCP -> Inductor_SMD:L_Bourns_SDR1806
- Q69: renamed from Q?; footprint Package_TO_SOT_THT:TO-220-3_Vertical -> Package_TO_SOT_SMD:TO-263-2
- gave numbers to parts that had none: 17
Connections:
- net +12V: now also U33.6 (Vin)
- net GND: now also U33.4 (GND)
- net HT: now also D2.1 (K)
- net at D1.2 (A), Q2.1 (B), R8.1: now also U33.2 (SwE)
- net at C37.1, L1.1, R3.1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: now also U33.1 (SwC), U33.7 (Ipk), U33.8 (DC)
- net at C16.1: now also U33.3 (TC)
- net at C38.2, R93.2, R94.1: now also U33.5 (Vfb)
- net at L1.2, Q69.2 (D): now also D2.2 (A)

Commit message: PCB rev2 layout in progress
Parts:
- C39: footprint Capacitor_THT:CP_Radial_D6.3mm_P2.50mm -> nixiedisp:CP_Radial_D6.3mm_P2.50mm_Horizontal
- U34: footprint Package_TO_SOT_THT:TO-220-3_Vertical -> Package_TO_SOT_SMD:TO-252-2
Connections:
- net TPAD: now reaches D2.2 (A), L1.2, Q69.2 (D)
Changed lines of the file:
@@
 AR Path="/60332D47/60380AC6" Ref="R8"  Part="1"
 F 0 "R8" H 5420 3896 50  0000 L CNN
-F 1 "1K" H 5420 3805 50  0000 L CNN
+F 1 "1K" V 5350 3800 50  0000 L CNN
 F 2 "Resistor_SMD:R_0805_2012Metric_Pad1.15x1.40mm_HandSolder" V 5280 3850 50  0001 C CNN
 F 3 "~" H 5350 3850 50  0001 C CNN
@@
 F 0 "C39" H 7165 3496 50  0000 L CNN
 F 1 "2.2uF 250V" H 7165 3405 50  0000 L CNN
-F 2 "Capacitor_THT:CP_Radial_D6.3mm_P2.50mm" H 7050 3450 50  0001 C CNN
+F 2 "nixiedisp:CP_Radial_D6.3mm_P2.50mm_Horizontal" H 7050 3450 50  0001 C CNN
 F 3 "~" H 7050 3450 50  0001 C CNN
 	1    7050 3450
@@
 F 0 "U34" H 4800 4792 50  0000 C CNN
 F 1 "L7805" H 4800 4701 50  0000 C CNN
-F 2 "Package_TO_SOT_THT:TO-220-3_Vertical" H 4825 4400 50  0001 L CIN
+F 2 "Package_TO_SOT_SMD:TO-252-2" H 4825 4400 50  0001 L CIN
 F 3 "http://www.st.com/content/ccc/resource/technical/document/datasheet/41/4f/b3/b0/12/d4/47/88/CD00000444.pdf/files/CD00000444.pdf/jcr:content/translations/en.CD00000444.pdf" H 4800 4500 50  0001 C CNN
 	1    4800 4550
@@
 Wire Wire Line
 	5200 3100 5200 3200
+Text Label 6150 3200 1    50   ~ 0
+TPAD
 $EndSCHEMATC
