File: hw/nixiedisp.kicad_pcb (KiCad board)
At the start: 2 copper layers, 140 x 94.1 mm, 222 parts, among them J1 serial port, J2 USB_B_Micro, J3 AVR-ISP-6, J4 12VDC IN, J5 HRLEDS, J6 pwr sw, Q1 MMBTA55, Q10 MMBTA42, Q11 MMBTA42, Q12 MMBTA42, Q13 MMBTA42, Q14 MMBTA42, Q15 MMBTA42, Q16 MMBTA42, Q17 MMBTA42, Q18 MMBTA42, Q19 MMBTA42, Q2 MMBTA55, Q20 MMBTA42, Q21 MMBTA42, Q22 MMBTA42, Q23 MMBTA42, Q24 MMBTA42, Q25 MMBTA42, Q26 MMBTA42, Q27 MMBTA42, Q28 MMBTA42, Q29 MMBTA42, Q3 MMBTA42, Q30 MMBTA42, Q31 MMBTA42, Q32 MMBTA42, Q33 MMBTA42, Q34 MMBTA42, Q35 MMBTA42, Q36 MMBTA42, Q37 MMBTA42, Q38 MMBTA42, Q39 MMBTA42, Q4 MMBTA42, Q40 MMBTA42, Q41 MMBTA42, Q42 MMBTA42, Q43 MMBTA42, Q44 MMBTA42, Q45 MMBTA42, Q46 MMBTA42, Q47 MMBTA42, Q48 MMBTA42, Q49 MMBTA42, Q5 MMBTA42, Q50 MMBTA42, Q51 MMBTA42, Q52 MMBTA42, Q53 MMBTA42, Q54 MMBTA42, Q55 MMBTA42, Q56 MMBTA42, Q57 MMBTA42, Q58 MMBTA42, Q59 MMBTA42, Q6 MMBTA42, Q60 MMBTA42, Q61 MMBTA42, Q62 MMBTA42, Q63 MMBTA42, Q64 MMBTA42, Q65 MMBTA42, Q66 MMBTA42, Q67 MMBTA42, Q68 MMBTA42, Q69 IRF740, Q7 MMBTA42, Q8 MMBTA42, Q9 MMBTA42, SW1 SW_MODE, SW2 SW_A, SW3 SW_B, U1 ATmega328P-AU, U10 IN14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

Commit message: rev2 board
Parts:
- added C17: 0.1uF, Capacitor_SMD:C_0805_2012Metric_Pad1.15x1.40mm_HandSolder, F.Cu at (188.1, 107.5)
- added G***: LOGO, nixiedisp:gnulogo, F.Cu at (141.9, 98.5)
- added H1: mounting hole, MountingHole:MountingHole_3.2mm_M3_Pad_Via, F.Cu at (73.0, 141.1)
- added H2: mounting hole, MountingHole:MountingHole_3.2mm_M3_Pad_Via, F.Cu at (73.0, 74.0)
- added H3: mounting hole, MountingHole:MountingHole_3.2mm_M3_Pad_Via, F.Cu at (204.0, 141.1)
- added H4: mounting hole, MountingHole:MountingHole_3.2mm_M3_Pad_Via, F.Cu at (204.0, 74.0)
- added J7: usbpwr, Connector_PinHeader_2.54mm:PinHeader_1x02_P2.54mm_Vertical, F.Cu at (127.2, 84.8)
- added R27: 10k, Resistor_SMD:R_0805_2012Metric_Pad1.15x1.40mm_HandSolder, B.Cu at (123.3, 84.8)
- added REF**: 12v DC, Symbol:Symbol_Barrel_Polarity, F.Cu at (95.0, 74.0)
- BT1, C10, C9: moved to F.Cu
- C18, C21, C24, C27, C30, C33, Y3: moved to B.Cu
- J3: value AVR-ISP-6 -> AVR-ISP
- SW1: value SW_MODE -> MODE
- SW2: value SW_A -> A
- SW3: value SW_B -> B
- moved J6 154.0 mm to (106.2, 87.0), turned to 180 degrees
- moved U34 146.8 mm to (116.2, 76.5), turned to 90 degrees
- moved BT1 129.3 mm to (167.9, 94.1), turned to 180 degrees
- moved C35 108.2 mm to (112.2, 85.0)
- moved Q1 102.7 mm to (149.3, 77.8)
- moved R1 102.7 mm to (152.7, 77.8)
- moved R2 102.7 mm to (155.2, 77.8)
- moved U3 102.7 mm to (151.8, 85.2)
- moved J1 102.5 mm to (189.0, 80.5)
- moved C36 101.4 mm to (120.3, 85.0), turned to 180 degrees
- moved J3 101.1 mm to (127.2, 77.3)
- moved C13 99.8 mm to (134.9, 85.5)
- moved C5 99.8 mm to (143.6, 77.5)
- moved C6 99.8 mm to (143.6, 80.0)
- moved U4 99.8 mm to (140.8, 85.5)
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Connections:
- J1 pad 1: (no net) -> Net-(J1-Pad1)
- J1 pad 4: (no net) -> Net-(J1-Pad4)
- J1 pad 6: (no net) -> Net-(J1-Pad6)
- J1 pad 9: (no net) -> Net-(J1-Pad9)
- J2 pad 4: (no net) -> Net-(J2-Pad4)
- U1 pad 19: (no net) -> Net-(U1-Pad19)
- U1 pad 20: (no net) -> Net-(U1-Pad20)
- U1 pad 22: (no net) -> Net-(U1-Pad22)
- U10 pad 13: (no net) -> Net-(U10-Pad13)
- U11 pad 13: (no net) -> Net-(U11-Pad13)
- U12 pad 13: (no net) -> Net-(U12-Pad13)
- U13 pad 13: (no net) -> Net-(U13-Pad13)
- U14 pad 13: (no net) -> Net-(U14-Pad13)
- U14 pad 14: (no net) -> Net-(U14-Pad14)
- U14 pad 15: (no net) -> Net-(U14-Pad15)
- U14 pad 16: (no net) -> Net-(U14-Pad16)
- U14 pad 19: (no net) -> Net-(U14-Pad19)
- U14 pad 20: (no net) -> Net-(U14-Pad20)
- U15 pad 13: (no net) -> Net-(U15-Pad13)
- U15 pad 14: (no net) -> Net-(U15-Pad14)
- U15 pad 15: (no net) -> Net-(U15-Pad15)
- U15 pad 16: (no net) -> Net-(U15-Pad16)
- U15 pad 19: (no net) -> Net-(U15-Pad19)
- U15 pad 20: (no net) -> Net-(U15-Pad20)
- U16 pad 13: (no net) -> Net-(U16-Pad13)
- U16 pad 14: (no net) -> Net-(U16-Pad14)
- U16 pad 15: (no net) -> Net-(U16-Pad15)
- U16 pad 16: (no net) -> Net-(U16-Pad16)
- U16 pad 19: (no net) -> Net-(U16-Pad19)
- U16 pad 20: (no net) -> Net-(U16-Pad20)
- U17 pad 13: (no net) -> Net-(U17-Pad13)
- U17 pad 14: (no net) -> Net-(U17-Pad14)
- U17 pad 15: (no net) -> Net-(U17-Pad15)
- U17 pad 16: (no net) -> Net-(U17-Pad16)
- U17 pad 19: (no net) -> Net-(U17-Pad19)
- U17 pad 20: (no net) -> Net-(U17-Pad20)
- U18 pad 13: (no net) -> Net-(U18-Pad13)
- U18 pad 14: (no net) -> Net-(U18-Pad14)
- U18 pad 15: (no net) -> Net-(U18-Pad15)
- U18 pad 16: (no net) -> Net-(U18-Pad16)
- U18 pad 19: (no net) -> Net-(U18-Pad19)
- U18 pad 20: (no net) -> Net-(U18-Pad20)
- U19 pad 13: (no net) -> Net-(U19-Pad13)
- U19 pad 14: (no net) -> Net-(U19-Pad14)
- U19 pad 15: (no net) -> Net-(U19-Pad15)
- U19 pad 16: (no net) -> Net-(U19-Pad16)
- U19 pad 19: (no net) -> Net-(U19-Pad19)
- U19 pad 20: (no net) -> Net-(U19-Pad20)
- U2 pad 9: (no net) -> Net-(U2-Pad9)
- U3 pad 11: (no net) -> Net-(U3-Pad11)
- U3 pad 8: (no net) -> Net-(U3-Pad8)
- U4 pad 10: (no net) -> Net-(U4-Pad10)
- U4 pad 2: (no net) -> Net-(U4-Pad2)
- U4 pad 3: (no net) -> Net-(U4-Pad3)
- U4 pad 7: (no net) -> Net-(U4-Pad7)
- U4 pad 8: (no net) -> Net-(U4-Pad8)
- U4 pad 9: (no net) -> Net-(U4-Pad9)
- U8 pad 13: (no net) -> Net-(U8-Pad13)
- U9 pad 13: (no net) -> Net-(U9-Pad13)
- Y3 pad 1: Net-(U32-Pad3) -> Net-(U32-Pad2)
- Y3 pad 2: Net-(U32-Pad2) -> Net-(U32-Pad3)
Routing:
- net VCC: track 59.1 -> 481.3 mm, vias 0 -> 16
- net GND: track 0.14 -> 155.8 mm, vias 0 -> 127
- net /TXD: track 3.62 -> 103.3 mm, vias 0 -> 2
- net /SCK: track 0.00 -> 71.3 mm, vias 0 -> 1
- net /MISO: track 0.00 -> 69.2 mm, vias 0 -> 1
- net /~RST: track 0.00 -> 68.2 mm, vias 0 -> 1
- net /RTC_CE: track 0.00 -> 65.6 mm, vias 0 -> 2
- net /RXD: track 0.00 -> 50.6 mm, vias 0 -> 2
- net /SRX: track 3.39 -> 51.7 mm
- net /ENUSB: track 3.06 -> 49.5 mm
- net /MOSI: track 0.00 -> 31.2 mm
- net /BDOT: track 51.3 -> 20.7 mm, vias 1 -> 3
- net /TX232: track 0.00 -> 25.9 mm
- net /SD: track 135.3 -> 160.3 mm
- net /VBATT: track 0.00 -> 24.7 mm
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- added copper zone on B.Cu, net /pwrsupply/TPAD
- added copper zone on F.Cu, net GND
Other:
- board size 140 x 94.1 mm -> 140 x 76.1 mm
- board text added: "All unmarked resistors: 47 kOhm All transistors: MMBTA42"
- board text added: "Don't populate both Y2 and Y3 they are alternative packages"
- board text removed: "Allakse to vreg se ksaploto, i akoma kalytera SMD"
- board text removed: "Allakse ton pyknoti se ksaploto (kai cutout sto PCB?)"
- board text removed: "Bottom half: - All unmarked resistors: 47 kOhm - All transistors: MMBTA42"
- board text removed: "CR2032"
- board text removed: "Cut along the line for a 4-digit display"
