File: hw/nixiedisp.sch (KiCad schematic (older format))
At the start: 48 parts, among them J1 serial port, J2 USB_B_Micro, J3 AVR-ISP-6, J5 HRLEDS, Q1 MMBTA55, U1 ATmega328P-AU, U10 IN14, U11 IN14, U12 IN14, U13 IN14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

Commit message: PCB rev2 layout in progress
Parts:
- added SW1: SW_MODE, nixiedisp:switch, symbol Switch:SW_Push
- added SW2: SW_A, nixiedisp:switch, symbol Switch:SW_Push
- added SW3: SW_B, nixiedisp:switch, symbol Switch:SW_Push
Connections:
- net GND: now also SW1.2, SW2.2, SW3.2
- net SWMODE: now reaches U1.26 (PC3)
- net SWMODE: now also SW1.1
- net SWA: now reaches U1.27 (PC4)
- net SWA: now also SW2.1
- net SWB: now reaches U1.28 (PC5)
- net SWB: now also SW3.1
- no-connect marks 27 -> 24
Other:
- moved on the sheet: J1, U5, U6

Commit message: rev2 board
Parts:
- added C17: 0.1uF, Capacitor_SMD:C_0805_2012Metric_Pad1.15x1.40mm_HandSolder, symbol Device:C_Small
- added H1, H2, H3, H4: mounting hole, MountingHole:MountingHole_3.2mm_M3_Pad_Via, symbol Mechanical:MountingHole_Pad
- added J7: usbpwr, Connector_PinHeader_2.54mm:PinHeader_1x02_P2.54mm_Vertical, symbol Connector_Generic:Conn_01x02
- added R27: 10k, Resistor_SMD:R_0805_2012Metric_Pad1.15x1.40mm_HandSolder, symbol Device:R
Connections:
- net ENUSB: now also J7.1 (Pin_1), R27.1
- net GND: now also C17.2, H1.1, H2.1, H3.1, H4.1, R27.2
- net VCC: now also C17.1, J7.2 (Pin_2)
- net at U32.2 (X1), Y2.1: now also Y3.1; no longer Y3.2
- net at U32.3 (X2), Y2.2: now also Y3.2; no longer Y3.1
Changed lines of the file:
@@
 L power:GND #PWR019
 U 1 1 61B0EE96
-P 3300 10950
-F 0 "#PWR019" H 3300 10700 50  0001 C CNN
-F 1 "GND" H 3300 10800 50  0000 C CNN
-F 2 "" H 3300 10950 50  0001 C CNN
-F 3 "" H 3300 10950 50  0001 C CNN
-	1    3300 10950
+P 3450 11000
+F 0 "#PWR019" H 3450 10750 50  0001 C CNN
+F 1 "GND" H 3450 10850 50  0000 C CNN
+F 2 "" H 3450 11000 50  0001 C CNN
+F 3 "" H 3450 11000 50  0001 C CNN
+	1    3450 11000
 	1    0    0    -1
 $EndComp
@@
 L power:VCC #PWR018
 U 1 1 61B3194F
-P 3300 10750
-F 0 "#PWR018" H 3300 10600 50  0001 C CNN
-F 1 "VCC" H 3300 10900 50  0000 C CNN
-F 2 "" H 3300 10750 50  0001 C CNN
-F 3 "" H 3300 10750 50  0001 C CNN
-	1    3300 10750
+P 3450 10700
+F 0 "#PWR018" H 3450 10550 50  0001 C CNN
+F 1 "VCC" H 3450 10850 50  0000 C CNN
+F 2 "" H 3450 10700 50  0001 C CNN
+F 3 "" H 3450 10700 50  0001 C CNN
+	1    3450 10700
 	1    0    0    -1
 $EndComp
@@
 F 4 "6pF" H 2450 1550 50  0001 C CNN "load"
 	1    2450 1550
-	0    -1   -1   0
+	0    -1   1    0
 $EndComp
 Connection ~ 2450 1450
@@
 	2550 7100 2550 7700
 Wire Wire Line
-	2550 7700 3450 7700
+	2550 7700 2900 7700
 Wire Wire Line
 	3750 7050 3800 7050
@@
 	3000 7350 3000 7050
 Wire Wire Line
-	650  7350 3000 7350
-Wire Wire Line
 	2450 6250 2450 7450
 Wire Wire Line
@@
 Connection ~ 2300 6150
 Wire Wire Line
-	1150 6050 1150 7700
+	1150 6050 1150 7250
 Wire Wire Line
 	1150 7700 2550 7700
@@
 Wire Wire Line
 	2050 3650 3350 3650
+$Comp
+L Mechanical:MountingHole_Pad H1
+U 1 1 600AE386
+P 9200 3050
+F 0 "H1" H 9150 3250 50  0000 L CNN
+F 1 "mounting hole" H 9250 3350 50  0000 L CNN
+F 2 "MountingHole:MountingHole_3.2mm_M3_Pad_Via" H 9200 3050 50  0001 C CNN
+F 3 "~" H 9200 3050 50  0001 C CNN
+	1    9200 3050
+	1    0    0    -1
+$EndComp
+Wire Wire Line
+	9200 3150 9400 3150
+$Comp
+L Mechanical:MountingHole_Pad H2
+U 1 1 600E222F
+P 9400 3050
+F 0 "H2" H 9350 3250 50  0000 L CNN
+F 1 "mounting hole" H 9500 3350 50  0001 L CNN
+F 2 "MountingHole:MountingHole_3.2mm_M3_Pad_Via" H 9400 3050 50  0001 C CNN
+F 3 "~" H 9400 3050 50  0001 C CNN
+	1    9400 3050
+	1    0    0    -1
+$EndComp
+Connection ~ 9400 3150
+Wire Wire Line
+	9400 3150 9500 3150
+$Comp
+L Mechanical:MountingHole_Pad H3
+U 1 1 600E2501
+P 9600 3050
+F 0 "H3" H 9550 3250 50  0000 L CNN
+F 1 "mounting hole" H 9700 3350 50  0001 L CNN
+F 2 "MountingHole:MountingHole_3.2mm_M3_Pad_Via" H 9600 3050 50  0001 C CNN
+F 3 "~" H 9600 3050 50  0001 C CNN
+	1    9600 3050
+	1    0    0    -1
+$EndComp
+Connection ~ 9600 3150
+Wire Wire Line
+	9600 3150 9800 3150
+$Comp
+L Mechanical:MountingHole_Pad H4
+U 1 1 600E27AD
+P 9800 3050
+F 0 "H4" H 9750 3250 50  0000 L CNN
+F 1 "mounting hole" H 9900 3350 50  0001 L CNN
+F 2 "MountingHole:MountingHole_3.2mm_M3_Pad_Via" H 9800 3050 50  0001 C CNN
+F 3 "~" H 9800 3050 50  0001 C CNN
+	1    9800 3050
+	1    0    0    -1
+$EndComp
+$Comp
+L power:GND #PWR045
+U 1 1 600E302B
+P 9500 3150
+F 0 "#PWR045" H 9500 2900 50  0001 C CNN
+F 1 "GND" H 9500 3000 50  0000 C CNN
+F 2 "" H 9500 3150 50  0001 C CNN
+F 3 "" H 9500 3150 50  0001 C CNN
+	1    9500 3150
+	1    0    0    -1
+$EndComp
+Connection ~ 9500 3150
+Wire Wire Line
+	9500 3150 9600 3150
+$Comp
+L Connector_Generic:Conn_01x02 J7
+U 1 1 60143D55
+P 700 7250
+AR Path="/60143D55" Ref="J7"  Part="1"
+AR Path="/60332D47/60143D55" Ref="J?"  Part="1"
+F 0 "J7" H 780 7242 50  0000 L CNN
+F 1 "usbpwr" H 600 7050 50  0000 L CNN
+F 2 "Connector_PinHeader_2.54mm:PinHeader_1x02_P2.54mm_Vertical" H 700 7250 50  0001 C CNN
+F 3 "~" H 700 7250 50  0001 C CNN
+	1    700  7250
+	-1   0    0    1
+$EndComp
+Wire Wire Line
+	650  7350 3000 7350
+Wire Wire Line
+	900  7250 1150 7250
+Connection ~ 1150 7250
+Wire Wire Line
+	1150 7250 1150 7700
+$Comp
+L power:VCC #PWR046
+U 1 1 60276A22
+P 900 7150
+F 0 "#PWR046" H 900 7000 50  0001 C CNN
+F 1 "VCC" H 900 7300 50  0000 C CNN
+F 2 "" H 900 7150 50  0001 C CNN
+F 3 "" H 900 7150 50  0001 C CNN
+	1    900  7150
+	1    0    0    -1
+$EndComp
+Connection ~ 3300 10950
+$Comp
+L Device:C_Small C17
+U 1 1 6032B882
+P 3300 10850
+F 0 "C17" H 3250 11000 50  0000 L CNN
+F 1 "0.1uF" H 3200 10700 50  0000 L CNN
+F 2 "Capacitor_SMD:C_0805_2012Metric_Pad1.15x1.40mm_HandSolder" H 3300 10850 50  0001 C CNN
+F 3 "~" H 3300 10850 50  0001 C CNN
+	1    3300 10850
+	1    0    0    -1
+$EndComp
+Wire Wire Line
+	3300 10950 3450 10950
+Wire Wire Line
+	3450 10950 3450 11000
+Wire Wire Line
+	3300 10750 3450 10750
+Wire Wire Line
+	3450 10750 3450 10700
+Connection ~ 3300 10750
+$Comp
+L Device:R R27
+U 1 1 60259940
+P 2900 7850
+F 0 "R27" V 2800 7850 50  0000 C CNN
+F 1 "10k" V 2900 7850 50  0000 C CNN
+F 2 "Resistor_SMD:R_0805_2012Metric_Pad1.15x1.40mm_HandSolder" V 2830 7850 50  0001 C CNN
+F 3 "~" H 2900 7850 50  0001 C CNN
+	1    2900 7850
+	-1   0    0    -1
+$EndComp
+Connection ~ 2900 7700
+Wire Wire Line
+	2900 7700 3450 7700
+$Comp
+L power:GND #PWR062
+U 1 1 6025A6DC
+P 2900 8000
+F 0 "#PWR062" H 2900 7750 50  0001 C CNN
+F 1 "GND" H 2900 7850 50  0000 C CNN
+F 2 "" H 2900 8000 50  0001 C CNN
+F 3 "" H 2900 8000 50  0001 C CNN
+	1    2900 8000
+	1    0    0    -1
+$EndComp
 $EndSCHEMATC
