File: hw/nixiedrivers.sch (KiCad schematic (older format))
At the start: 30 parts, among them Q10 MMBTA42, Q11 MMBTA42, Q12 MMBTA42, Q13 MMBTA42, Q3 MMBTA42, Q4 MMBTA42, Q5 MMBTA42, Q6 MMBTA42, Q7 MMBTA42, Q8 MMBTA42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

Commit message: lots of changes, redesigning most of the PCB
Parts:
- removed C17, C19: 0.1uF, Capacitor_SMD:C_0805_2012Metric_Pad1.15x1.40mm_HandSolder, symbol Device:C
- removed R27: 47k, Resistor_SMD:R_0805_2012Metric_Pad1.15x1.40mm_HandSolder, symbol Device:R
- removed U14: 74HC154, Package_SO:SOIC-24W_7.5x15.4mm_P1.27mm, symbol 74xx:74LS154
- removed U15, U16: 74HC04, Package_SO:SO-14_5.3x10.2mm_P1.27mm, symbol 74xx:74HC04
- added U14: 74HC4514, Package_SO:SOIC-24W_7.5x15.4mm_P1.27mm, symbol 4xxx_IEEE:4514
- R21: value 47k -> 160k
Connections:
- net D0: now also U14.2 (A0)
- net D1: now also U14.3 (A1)
- net D2: now also U14.21 (A2)
- net D3: now also U14.22 (A3)
- net GND: now also U14.12 (Vss), U14.23 (~EN)
- net NL: now also R21.1
- net VCC: now also U14.1 (EL), U14.24 (Vdd)
- net at R15.2: now also U14.11 (Q0)
- net at R22.2: now also U14.9 (Q1)
- net at R16.2: now also U14.10 (Q2)
- net at R23.2: now also U14.8 (Q3)
- net at R17.2: now also U14.7 (Q4)
- net at R24.2: now also U14.6 (Q5)
- net at R18.2: now also U14.5 (Q6)
- net at R25.2: now also U14.4 (Q7)
- net at R19.2: now also U14.18 (Q8)
- net at R26.2: now also U14.17 (Q9)
- no-connect marks 8 -> 6
Other:
- moved on the sheet: C33

Commit message: PCB rev2 layout in progress
Changed lines of the file:
@@
 $Descr A4 11693 8268
 encoding utf-8
-Sheet 7 8
+Sheet 3 8
 Title "USB nixie tube display"
 Date "2021-01-19"
@@
 AR Path="/603FFB52/5FF0530D" Ref="Q36"  Part="1"
 AR Path="/603FFDD2/5FF0530D" Ref="Q47"  Part="1"
-F 0 "Q58" H 5200 1350 50  0000 L CNN
+F 0 "Q14" H 5200 1350 50  0000 L CNN
 F 1 "MMBTA42" H 5100 1650 50  0000 L CNN
 F 2 "Package_TO_SOT_SMD:SOT-23" H 5550 1425 50  0001 L CIN
@@
 AR Path="/603FFB52/5FF05313" Ref="R54"  Part="1"
 AR Path="/603FFDD2/5FF05313" Ref="R67"  Part="1"
-F 0 "R80" V 4850 1500 50  0000 C CNN
+F 0 "R28" V 4850 1500 50  0000 C CNN
 F 1 "47k" V 4950 1500 50  0000 C CNN
 F 2 "Resistor_SMD:R_0805_2012Metric_Pad1.15x1.40mm_HandSolder" V 4880 1500 50  0001 C CNN
@@
 AR Path="/603FFB52/5FF05321" Ref="Q42"  Part="1"
 AR Path="/603FFDD2/5FF05321" Ref="Q53"  Part="1"
-F 0 "Q64" H 6000 1800 50  0000 L CNN
+F 0 "Q20" H 6000 1800 50  0000 L CNN
 F 1 "MMBTA42" H 5900 2100 50  0000 L CNN
 F 2 "Package_TO_SOT_SMD:SOT-23" H 6350 1875 50  0001 L CIN
@@
 AR Path="/603FFB52/5FF05327" Ref="R61"  Part="1"
 AR Path="/603FFDD2/5FF05327" Ref="R74"  Part="1"
-F 0 "R87" V 5650 1950 50  0000 C CNN
+F 0 "R35" V 5650 1950 50  0000 C CNN
 F 1 "47k" V 5750 1950 50  0000 C CNN
 F 2 "Resistor_SMD:R_0805_2012Metric_Pad1.15x1.40mm_HandSolder" V 5680 1950 50  0001 C CNN
@@
 AR Path="/603FFB52/5FF07144" Ref="Q37"  Part="1"
 AR Path="/603FFDD2/5FF07144" Ref="Q48"  Part="1"
-F 0 "Q59" H 5200 2150 50  0000 L CNN
+F 0 "Q15" H 5200 2150 50  0000 L CNN
 F 1 "MMBTA42" H 5100 2450 50  0000 L CNN
 F 2 "Package_TO_SOT_SMD:SOT-23" H 5550 2225 50  0001 L CIN
@@
 AR Path="/603FFB52/5FF071D6" Ref="R55"  Part="1"
 AR Path="/603FFDD2/5FF071D6" Ref="R68"  Part="1"
-F 0 "R81" V 4850 2300 50  0000 C CNN
+F 0 "R29" V 4850 2300 50  0000 C CNN
 F 1 "47k" V 4950 2300 50  0000 C CNN
 F 2 "Resistor_SMD:R_0805_2012Metric_Pad1.15x1.40mm_HandSolder" V 4880 2300 50  0001 C CNN
@@
 AR Path="/603FFB52/5FF071EC" Ref="Q43"  Part="1"
 AR Path="/603FFDD2/5FF071EC" Ref="Q54"  Part="1"
-F 0 "Q65" H 6000 2600 50  0000 L CNN
+F 0 "Q21" H 6000 2600 50  0000 L CNN
 F 1 "MMBTA42" H 5900 2900 50  0000 L CNN
 F 2 "Package_TO_SOT_SMD:SOT-23" H 6350 2675 50  0001 L CIN
@@
 AR Path="/603FFB52/5FF071F6" Ref="R62"  Part="1"
 AR Path="/603FFDD2/5FF071F6" Ref="R75"  Part="1"
-F 0 "R88" V 5650 2750 50  0000 C CNN
+F 0 "R36" V 5650 2750 50  0000 C CNN
 F 1 "47k" V 5750 2750 50  0000 C CNN
 F 2 "Resistor_SMD:R_0805_2012Metric_Pad1.15x1.40mm_HandSolder" V 5680 2750 50  0001 C CNN
@@
 AR Path="/603FFB52/5FF09C0A" Ref="Q38"  Part="1"
 AR Path="/603FFDD2/5FF09C0A" Ref="Q49"  Part="1"
-F 0 "Q60" H 5200 2950 50  0000 L CNN
+F 0 "Q16" H 5200 2950 50  0000 L CNN
 F 1 "MMBTA42" H 5100 3250 50  0000 L CNN
 F 2 "Package_TO_SOT_SMD:SOT-23" H 5550 3025 50  0001 L CIN
@@
 AR Path="/603FFB52/5FF09D0C" Ref="R56"  Part="1"
 AR Path="/603FFDD2/5FF09D0C" Ref="R69"  Part="1"
-F 0 "R82" V 4850 3100 50  0000 C CNN
+F 0 "R30" V 4850 3100 50  0000 C CNN
 F 1 "47k" V 4950 3100 50  0000 C CNN
 F 2 "Resistor_SMD:R_0805_2012Metric_Pad1.15x1.40mm_HandSolder" V 4880 3100 50  0001 C CNN
@@
 AR Path="/603FFB52/5FF09D22" Ref="Q44"  Part="1"
 AR Path="/603FFDD2/5FF09D22" Ref="Q55"  Part="1"
-F 0 "Q66" H 6000 3400 50  0000 L CNN
+F 0 "Q22" H 6000 3400 50  0000 L CNN
 F 1 "MMBTA42" H 5900 3700 50  0000 L CNN
 F 2 "Package_TO_SOT_SMD:SOT-23" H 6350 3475 50  0001 L CIN
@@
 AR Path="/603FFB52/5FF09D2C" Ref="R63"  Part="1"
 AR Path="/603FFDD2/5FF09D2C" Ref="R76"  Part="1"
-F 0 "R89" V 5650 3550 50  0000 C CNN
+F 0 "R37" V 5650 3550 50  0000 C CNN
 F 1 "47k" V 5750 3550 50  0000 C CNN
 F 2 "Resistor_SMD:R_0805_2012Metric_Pad1.15x1.40mm_HandSolder" V 5680 3550 50  0001 C CNN
@@
 AR Path="/603FFB52/5FF09D42" Ref="Q39"  Part="1"
 AR Path="/603FFDD2/5FF09D42" Ref="Q50"  Part="1"
-F 0 "Q61" H 5200 3750 50  0000 L CNN
+F 0 "Q17" H 5200 3750 50  0000 L CNN
 F 1 "MMBTA42" H 5100 4050 50  0000 L CNN
 F 2 "Package_TO_SOT_SMD:SOT-23" H 5550 3825 50  0001 L CIN
@@
 AR Path="/603FFB52/5FF09D4C" Ref="R57"  Part="1"
 AR Path="/603FFDD2/5FF09D4C" Ref="R70"  Part="1"
-F 0 "R83" V 4850 3900 50  0000 C CNN
+F 0 "R31" V 4850 3900 50  0000 C CNN
 F 1 "47k" V 4950 3900 50  0000 C CNN
 F 2 "Resistor_SMD:R_0805_2012Metric_Pad1.15x1.40mm_HandSolder" V 4880 3900 50  0001 C CNN
@@
 AR Path="/603FFB52/5FF09D62" Ref="Q45"  Part="1"
 AR Path="/603FFDD2/5FF09D62" Ref="Q56"  Part="1"
-F 0 "Q67" H 6000 4200 50  0000 L CNN
+F 0 "Q23" H 6000 4200 50  0000 L CNN
 F 1 "MMBTA42" H 5900 4500 50  0000 L CNN
 F 2 "Package_TO_SOT_SMD:SOT-23" H 6350 4275 50  0001 L CIN
@@
 AR Path="/603FFB52/5FF09D6C" Ref="R64"  Part="1"
 AR Path="/603FFDD2/5FF09D6C" Ref="R77"  Part="1"
-F 0 "R90" V 5650 4350 50  0000 C CNN
+F 0 "R38" V 5650 4350 50  0000 C CNN
 F 1 "47k" V 5750 4350 50  0000 C CNN
 F 2 "Resistor_SMD:R_0805_2012Metric_Pad1.15x1.40mm_HandSolder" V 5680 4350 50  0001 C CNN
@@
 AR Path="/603FFB52/5FF15CE1" Ref="Q40"  Part="1"
 AR Path="/603FFDD2/5FF15CE1" Ref="Q51"  Part="1"
-F 0 "Q62" H 5200 4550 50  0000 L CNN
+F 0 "Q18" H 5200 4550 50  0000 L CNN
 F 1 "MMBTA42" H 5100 4850 50  0000 L CNN
 F 2 "Package_TO_SOT_SMD:SOT-23" H 5550 4625 50  0001 L CIN
@@
 AR Path="/603FFB52/5FF15EC3" Ref="R58"  Part="1"
 AR Path="/603FFDD2/5FF15EC3" Ref="R71"  Part="1"
-F 0 "R84" V 4850 4700 50  0000 C CNN
+F 0 "R32" V 4850 4700 50  0000 C CNN
 F 1 "47k" V 4950 4700 50  0000 C CNN
 F 2 "Resistor_SMD:R_0805_2012Metric_Pad1.15x1.40mm_HandSolder" V 4880 4700 50  0001 C CNN
@@
 AR Path="/603FFB52/5FF15ED9" Ref="Q46"  Part="1"
 AR Path="/603FFDD2/5FF15ED9" Ref="Q57"  Part="1"
-F 0 "Q68" H 6000 5000 50  0000 L CNN
+F 0 "Q24" H 6000 5000 50  0000 L CNN
 F 1 "MMBTA42" H 5900 5300 50  0000 L CNN
 F 2 "Package_TO_SOT_SMD:SOT-23" H 6350 5075 50  0001 L CIN
@@
 AR Path="/603FFB52/5FF15EE3" Ref="R65"  Part="1"
 AR Path="/603FFDD2/5FF15EE3" Ref="R78"  Part="1"
-F 0 "R91" V 5650 5150 50  0000 C CNN
+F 0 "R39" V 5650 5150 50  0000 C CNN
 F 1 "47k" V 5750 5150 50  0000 C CNN
 F 2 "Resistor_SMD:R_0805_2012Metric_Pad1.15x1.40mm_HandSolder" V 5680 5150 50  0001 C CNN
@@
 AR Path="/603FFB52/5FF15EF9" Ref="Q41"  Part="1"
 AR Path="/603FFDD2/5FF15EF9" Ref="Q52"  Part="1"
-F 0 "Q63" H 5200 5700 50  0000 L CNN
+F 0 "Q19" H 5200 5700 50  0000 L CNN
 F 1 "MMBTA42" H 5100 6000 50  0000 L CNN
 F 2 "Package_TO_SOT_SMD:SOT-23" H 5550 5775 50  0001 L CIN
@@
 AR Path="/603FFB52/5FF15F03" Ref="R59"  Part="1"
 AR Path="/603FFDD2/5FF15F03" Ref="R72"  Part="1"
-F 0 "R85" V 4850 5850 50  0000 C CNN
+F 0 "R33" V 4850 5850 50  0000 C CNN
 F 1 "47k" V 4950 5850 50  0000 C CNN
 F 2 "Resistor_SMD:R_0805_2012Metric_Pad1.15x1.40mm_HandSolder" V 4880 5850 50  0001 C CNN
@@
 AR Path="/603FFB52/5FF51489" Ref="R60"  Part="1"
 AR Path="/603FFDD2/5FF51489" Ref="R73"  Part="1"
-F 0 "R86" V 5600 5650 50  0000 C CNN
+F 0 "R34" V 5600 5650 50  0000 C CNN
 F 1 "160k" V 5700 5650 50  0000 C CNN
 F 2 "Resistor_SMD:R_0805_2012Metric_Pad1.15x1.40mm_HandSolder" V 5630 5650 50  0001 C CNN
@@
 AR Path="/603FFDD2/61F3B605" Ref="C30"  Part="1"
 AR Path="/603EFAE2/61F3B605" Ref="C33"  Part="1"
-F 0 "C33" H 3350 5000 50  0000 L CNN
+F 0 "C21" H 3350 5000 50  0000 L CNN
 F 1 "0.1uF" H 3350 4800 50  0000 L CNN
 F 2 "Capacitor_SMD:C_0805_2012Metric_Pad1.15x1.40mm_HandSolder" H 3338 4750 50  0001 C CNN
@@
 AR Path="/603FFDD2/62811958" Ref="U18"  Part="1"
 AR Path="/603EFAE2/62811958" Ref="U19"  Part="1"
-F 0 "U19" H 3450 4300 50  0000 C CNN
+F 0 "U15" H 3450 4300 50  0000 C CNN
 F 1 "74HC4514" H 3550 4200 50  0000 C CNN
 F 2 "Package_SO:SOIC-24W_7.5x15.4mm_P1.27mm" H 3300 3350 50  0001 C CNN

Commit message: rev2 board
Changed lines of the file:
@@
 $Descr A4 11693 8268
 encoding utf-8
-Sheet 3 8
+Sheet 6 8
 Title "USB nixie tube display"
 Date "2021-01-19"
@@
 AR Path="/603FFB52/5FF0530D" Ref="Q36"  Part="1"
 AR Path="/603FFDD2/5FF0530D" Ref="Q47"  Part="1"
-F 0 "Q14" H 5200 1350 50  0000 L CNN
+F 0 "Q58" H 5200 1350 50  0000 L CNN
 F 1 "MMBTA42" H 5100 1650 50  0000 L CNN
 F 2 "Package_TO_SOT_SMD:SOT-23" H 5550 1425 50  0001 L CIN
@@
 AR Path="/603FFB52/5FF05313" Ref="R54"  Part="1"
 AR Path="/603FFDD2/5FF05313" Ref="R67"  Part="1"
-F 0 "R28" V 4850 1500 50  0000 C CNN
+F 0 "R80" V 4850 1500 50  0000 C CNN
 F 1 "47k" V 4950 1500 50  0000 C CNN
 F 2 "Resistor_SMD:R_0805_2012Metric_Pad1.15x1.40mm_HandSolder" V 4880 1500 50  0001 C CNN
@@
 AR Path="/603FFB52/5FF05321" Ref="Q42"  Part="1"
 AR Path="/603FFDD2/5FF05321" Ref="Q53"  Part="1"
-F 0 "Q20" H 6000 1800 50  0000 L CNN
+F 0 "Q64" H 6000 1800 50  0000 L CNN
 F 1 "MMBTA42" H 5900 2100 50  0000 L CNN
 F 2 "Package_TO_SOT_SMD:SOT-23" H 6350 1875 50  0001 L CIN
@@
 AR Path="/603FFB52/5FF05327" Ref="R61"  Part="1"
 AR Path="/603FFDD2/5FF05327" Ref="R74"  Part="1"
-F 0 "R35" V 5650 1950 50  0000 C CNN
+F 0 "R87" V 5650 1950 50  0000 C CNN
 F 1 "47k" V 5750 1950 50  0000 C CNN
 F 2 "Resistor_SMD:R_0805_2012Metric_Pad1.15x1.40mm_HandSolder" V 5680 1950 50  0001 C CNN
@@
 AR Path="/603FFB52/5FF07144" Ref="Q37"  Part="1"
 AR Path="/603FFDD2/5FF07144" Ref="Q48"  Part="1"
-F 0 "Q15" H 5200 2150 50  0000 L CNN
+F 0 "Q59" H 5200 2150 50  0000 L CNN
 F 1 "MMBTA42" H 5100 2450 50  0000 L CNN
 F 2 "Package_TO_SOT_SMD:SOT-23" H 5550 2225 50  0001 L CIN
@@
 AR Path="/603FFB52/5FF071D6" Ref="R55"  Part="1"
 AR Path="/603FFDD2/5FF071D6" Ref="R68"  Part="1"
-F 0 "R29" V 4850 2300 50  0000 C CNN
+F 0 "R81" V 4850 2300 50  0000 C CNN
 F 1 "47k" V 4950 2300 50  0000 C CNN
 F 2 "Resistor_SMD:R_0805_2012Metric_Pad1.15x1.40mm_HandSolder" V 4880 2300 50  0001 C CNN
@@
 AR Path="/603FFB52/5FF071EC" Ref="Q43"  Part="1"
 AR Path="/603FFDD2/5FF071EC" Ref="Q54"  Part="1"
-F 0 "Q21" H 6000 2600 50  0000 L CNN
+F 0 "Q65" H 6000 2600 50  0000 L CNN
 F 1 "MMBTA42" H 5900 2900 50  0000 L CNN
 F 2 "Package_TO_SOT_SMD:SOT-23" H 6350 2675 50  0001 L CIN
@@
 AR Path="/603FFB52/5FF071F6" Ref="R62"  Part="1"
 AR Path="/603FFDD2/5FF071F6" Ref="R75"  Part="1"
-F 0 "R36" V 5650 2750 50  0000 C CNN
+F 0 "R88" V 5650 2750 50  0000 C CNN
 F 1 "47k" V 5750 2750 50  0000 C CNN
 F 2 "Resistor_SMD:R_0805_2012Metric_Pad1.15x1.40mm_HandSolder" V 5680 2750 50  0001 C CNN
@@
 AR Path="/603FFB52/5FF09C0A" Ref="Q38"  Part="1"
 AR Path="/603FFDD2/5FF09C0A" Ref="Q49"  Part="1"
-F 0 "Q16" H 5200 2950 50  0000 L CNN
+F 0 "Q60" H 5200 2950 50  0000 L CNN
 F 1 "MMBTA42" H 5100 3250 50  0000 L CNN
 F 2 "Package_TO_SOT_SMD:SOT-23" H 5550 3025 50  0001 L CIN
@@
 AR Path="/603FFB52/5FF09D0C" Ref="R56"  Part="1"
 AR Path="/603FFDD2/5FF09D0C" Ref="R69"  Part="1"
-F 0 "R30" V 4850 3100 50  0000 C CNN
+F 0 "R82" V 4850 3100 50  0000 C CNN
 F 1 "47k" V 4950 3100 50  0000 C CNN
 F 2 "Resistor_SMD:R_0805_2012Metric_Pad1.15x1.40mm_HandSolder" V 4880 3100 50  0001 C CNN
@@
 AR Path="/603FFB52/5FF09D22" Ref="Q44"  Part="1"
 AR Path="/603FFDD2/5FF09D22" Ref="Q55"  Part="1"
-F 0 "Q22" H 6000 3400 50  0000 L CNN
+F 0 "Q66" H 6000 3400 50  0000 L CNN
 F 1 "MMBTA42" H 5900 3700 50  0000 L CNN
 F 2 "Package_TO_SOT_SMD:SOT-23" H 6350 3475 50  0001 L CIN
@@
 AR Path="/603FFB52/5FF09D2C" Ref="R63"  Part="1"
 AR Path="/603FFDD2/5FF09D2C" Ref="R76"  Part="1"
-F 0 "R37" V 5650 3550 50  0000 C CNN
+F 0 "R89" V 5650 3550 50  0000 C CNN
 F 1 "47k" V 5750 3550 50  0000 C CNN
 F 2 "Resistor_SMD:R_0805_2012Metric_Pad1.15x1.40mm_HandSolder" V 5680 3550 50  0001 C CNN
@@
 AR Path="/603FFB52/5FF09D42" Ref="Q39"  Part="1"
 AR Path="/603FFDD2/5FF09D42" Ref="Q50"  Part="1"
-F 0 "Q17" H 5200 3750 50  0000 L CNN
+F 0 "Q61" H 5200 3750 50  0000 L CNN
 F 1 "MMBTA42" H 5100 4050 50  0000 L CNN
 F 2 "Package_TO_SOT_SMD:SOT-23" H 5550 3825 50  0001 L CIN
@@
 AR Path="/603FFB52/5FF09D4C" Ref="R57"  Part="1"
 AR Path="/603FFDD2/5FF09D4C" Ref="R70"  Part="1"
-F 0 "R31" V 4850 3900 50  0000 C CNN
+F 0 "R83" V 4850 3900 50  0000 C CNN
 F 1 "47k" V 4950 3900 50  0000 C CNN
 F 2 "Resistor_SMD:R_0805_2012Metric_Pad1.15x1.40mm_HandSolder" V 4880 3900 50  0001 C CNN
@@
 AR Path="/603FFB52/5FF09D62" Ref="Q45"  Part="1"
 AR Path="/603FFDD2/5FF09D62" Ref="Q56"  Part="1"
-F 0 "Q23" H 6000 4200 50  0000 L CNN
+F 0 "Q67" H 6000 4200 50  0000 L CNN
 F 1 "MMBTA42" H 5900 4500 50  0000 L CNN
 F 2 "Package_TO_SOT_SMD:SOT-23" H 6350 4275 50  0001 L CIN
@@
 AR Path="/603FFB52/5FF09D6C" Ref="R64"  Part="1"
 AR Path="/603FFDD2/5FF09D6C" Ref="R77"  Part="1"
-F 0 "R38" V 5650 4350 50  0000 C CNN
+F 0 "R90" V 5650 4350 50  0000 C CNN
 F 1 "47k" V 5750 4350 50  0000 C CNN
 F 2 "Resistor_SMD:R_0805_2012Metric_Pad1.15x1.40mm_HandSolder" V 5680 4350 50  0001 C CNN
@@
 AR Path="/603FFB52/5FF15CE1" Ref="Q40"  Part="1"
 AR Path="/603FFDD2/5FF15CE1" Ref="Q51"  Part="1"
-F 0 "Q18" H 5200 4550 50  0000 L CNN
+F 0 "Q62" H 5200 4550 50  0000 L CNN
 F 1 "MMBTA42" H 5100 4850 50  0000 L CNN
 F 2 "Package_TO_SOT_SMD:SOT-23" H 5550 4625 50  0001 L CIN
@@
 AR Path="/603FFB52/5FF15EC3" Ref="R58"  Part="1"
 AR Path="/603FFDD2/5FF15EC3" Ref="R71"  Part="1"
-F 0 "R32" V 4850 4700 50  0000 C CNN
+F 0 "R84" V 4850 4700 50  0000 C CNN
 F 1 "47k" V 4950 4700 50  0000 C CNN
 F 2 "Resistor_SMD:R_0805_2012Metric_Pad1.15x1.40mm_HandSolder" V 4880 4700 50  0001 C CNN
@@
 AR Path="/603FFB52/5FF15ED9" Ref="Q46"  Part="1"
 AR Path="/603FFDD2/5FF15ED9" Ref="Q57"  Part="1"
-F 0 "Q24" H 6000 5000 50  0000 L CNN
+F 0 "Q68" H 6000 5000 50  0000 L CNN
 F 1 "MMBTA42" H 5900 5300 50  0000 L CNN
 F 2 "Package_TO_SOT_SMD:SOT-23" H 6350 5075 50  0001 L CIN
@@
 AR Path="/603FFB52/5FF15EE3" Ref="R65"  Part="1"
 AR Path="/603FFDD2/5FF15EE3" Ref="R78"  Part="1"
-F 0 "R39" V 5650 5150 50  0000 C CNN
+F 0 "R91" V 5650 5150 50  0000 C CNN
 F 1 "47k" V 5750 5150 50  0000 C CNN
 F 2 "Resistor_SMD:R_0805_2012Metric_Pad1.15x1.40mm_HandSolder" V 5680 5150 50  0001 C CNN
@@
 AR Path="/603FFB52/5FF15EF9" Ref="Q41"  Part="1"
 AR Path="/603FFDD2/5FF15EF9" Ref="Q52"  Part="1"
-F 0 "Q19" H 5200 5700 50  0000 L CNN
+F 0 "Q63" H 5200 5700 50  0000 L CNN
 F 1 "MMBTA42" H 5100 6000 50  0000 L CNN
 F 2 "Package_TO_SOT_SMD:SOT-23" H 5550 5775 50  0001 L CIN
@@
 AR Path="/603FFB52/5FF15F03" Ref="R59"  Part="1"
 AR Path="/603FFDD2/5FF15F03" Ref="R72"  Part="1"
-F 0 "R33" V 4850 5850 50  0000 C CNN
+F 0 "R85" V 4850 5850 50  0000 C CNN
 F 1 "47k" V 4950 5850 50  0000 C CNN
 F 2 "Resistor_SMD:R_0805_2012Metric_Pad1.15x1.40mm_HandSolder" V 4880 5850 50  0001 C CNN
@@
 AR Path="/603FFB52/5FF51489" Ref="R60"  Part="1"
 AR Path="/603FFDD2/5FF51489" Ref="R73"  Part="1"
-F 0 "R34" V 5600 5650 50  0000 C CNN
+F 0 "R86" V 5600 5650 50  0000 C CNN
 F 1 "160k" V 5700 5650 50  0000 C CNN
 F 2 "Resistor_SMD:R_0805_2012Metric_Pad1.15x1.40mm_HandSolder" V 5630 5650 50  0001 C CNN
@@
 AR Path="/603FFDD2/61F3B605" Ref="C30"  Part="1"
 AR Path="/603EFAE2/61F3B605" Ref="C33"  Part="1"
-F 0 "C21" H 3350 5000 50  0000 L CNN
+F 0 "C33" H 3350 5000 50  0000 L CNN
 F 1 "0.1uF" H 3350 4800 50  0000 L CNN
 F 2 "Capacitor_SMD:C_0805_2012Metric_Pad1.15x1.40mm_HandSolder" H 3338 4750 50  0001 C CNN
@@
 AR Path="/603FFDD2/62811958" Ref="U18"  Part="1"
 AR Path="/603EFAE2/62811958" Ref="U19"  Part="1"
-F 0 "U15" H 3450 4300 50  0000 C CNN
+F 0 "U19" H 3450 4300 50  0000 C CNN
 F 1 "74HC4514" H 3550 4200 50  0000 C CNN
 F 2 "Package_SO:SOIC-24W_7.5x15.4mm_P1.27mm" H 3300 3350 50  0001 C CNN
